Commit message: adding steering pivot point

File: src/ros_controllers/four_wheel_steering_controller/test/urdf/four_wheel_steering.urdf.xacro (robot description, xacro)
@@ -7,5 +7,5 @@
   <xacro:property name="ground_clearance" value="0.19" />
   <xacro:property name="wheel_x_offset" value="0.0" />
-  <xacro:property name="wheel_y_offset" value="0.05" />
+  <xacro:property name="wheel_y_offset" value="0.1" />
   <xacro:chassis/>
   <!-- Wheel macros -->

File: src/ros_controllers/four_wheel_steering_controller/test/urdf/wheel.xacro (robot description, xacro)
@@ -38,6 +38,6 @@
 		</link>
 		<gazebo reference="${wheel_prefix}_wheel_link">
-			<mu1 value="1.0"/>
-			<mu2 value="1.0"/>
+			<mu1 value="0.1"/>
+			<mu2 value="0.1"/>
 			<kp value="10000000.0" />
 			<kd value="1.0" />
