Commit message: adding joystick

File: src/ros_controllers/four_wheel_steering_controller/test/urdf/chassis.xacro (robot description, xacro)
@@ -1,904 +1,54 @@
 <?xml version="1.0"?>
-<!--
-Software License Agreement (BSD License)
-Copyright (c) 2020, Exobotic
-All rights reserved.
-Redistribution and use in source and binary forms, with or without
-modification, are permitted provided that the following conditions
-are met:
- * Redistributions of source code must retain the above copyright
-   notice, this list of conditions and the following disclaimer.
- * Redistributions in binary form must reproduce the above
-   copyright notice, this list of conditions and the following
-   disclaimer in the documentation and/or other materials provided
-   with the distribution.
- * Neither the name of Exobotic nor the names of its
-   contributors may be used to endorse or promote products derived
-   from this software without specific prior written permission.
-THIS SOFTWARE IS PROVIDED BY THE COPYRIGHT HOLDERS AND CONTRIBUTORS
-"AS IS" AND ANY EXPRESS OR IMPLIED WARRANTIES, INCLUDING, BUT NOT
-LIMITED TO, THE IMPLIED WARRANTIES OF MERCHANTABILITY AND FITNESS
-FOR A PARTICULAR PURPOSE ARE DISCLAIMED. IN NO EVENT SHALL THE
-COPYRIGHT OWNER OR CONTRIBUTORS BE LIABLE FOR ANY DIRECT, INDIRECT,
-INCIDENTAL, SPECIAL, EXEMPLARY, OR CONSEQUENTIAL DAMAGES (INCLUDING,
-BUT NOT LIMITED TO, PROCUREMENT OF SUBSTITUTE GOODS OR SERVICES;
-LOSS OF USE, DATA, OR PROFITS; OR BUSINESS INTERRUPTION) HOWEVER
-CAUSED AND ON ANY THEORY OF LIABILITY, WHETHER IN CONTRACT, STRICT
-LIABILITY, OR TORT (INCLUDING NEGLIGENCE OR OTHERWISE) ARISING IN
-ANY WAY OUT OF THE USE OF THIS SOFTWARE, EVEN IF ADVISED OF THE
-POSSIBILITY OF SUCH DAMAGE.
--->
-<!-- created with Phobos 1.0.1 "Capricious Choutengan" -->
-  <robot name="m2"
-         xmlns:xacro="http://www.ros.org/wiki/xacro">
-    <material name="LiDAR_grey">
-      <color rgba="0.59608 0.59608 0.59608 1.0"/>
-    </material>
-    <material name="Metal_Bling chrome">
-      <color rgba="0.8 0.8 0.82431 1.0"/>
-    </material>
-    <material name="Synth_Tyre rubber">
-      <color rgba="0.01678 0.01212 0.01212 1.0"/>
-    </material>
-    <material name="blue_police_light">
-      <color rgba="0 0 1.0 1.0"/>
-    </material>
-    <material name="body_black">
-      <color rgba="0.10594 0.10594 0.10594 1.0"/>
-    </material>
-    <material name="body_grey">
-      <color rgba="0.96 0.96 0.96 1.0"/>
-    </material>
-    <material name="red_police_light">
-      <color rgba="1.0 0 0 1.0"/>
-    </material>
-    <material name="white_police_light">
-      <color rgba="1.0 1.0 1.0 1.0"/>
-    </material>
-    <material name="dummy_mat">
-      <color rgba="0.4 0.4 0.4 1.0"/>
-    </material>
+<robot xmlns:xacro="http://www.ros.org/wiki/xacro" name="chassis">
+  <!-- Base Properties -->
+  <xacro:property name="mass_base" value="340" />
+  <xacro:property name="base_x_size" value="1.66000" />
+  <xacro:property name="base_y_size" value="0.60000" />
+  <xacro:property name="base_z_size" value="0.66000" />
+  <xacro:property name="wheelbase" value="1.9" />
+  <xacro:property name="track" value="1.1" />
+  <xacro:macro name="chassis">
+    <!-- Base footprint is on the ground under the robot -->
     <link name="base_footprint"/>
-    <link name="chassis">
-      <inertial>
-        <origin xyz="0.08838 -0.00198 0.17552" rpy="0 0 0"/>
-        <mass value="200.0"/>
-        <inertia ixx="24.43942" ixy="-3.57208" ixz="-2.64293" iyy="116.11656" iyz="0.10486" izz="111.43803"/>
-      </inertial>
-      <visual name="body_front_lights_vis">
-        <origin xyz="0.98421 0.00023 0.09713" rpy="0 0 0"/>
+    <gazebo reference="base_link">
+      <material>Gazebo/Grey</material>
+    </gazebo>
+    <!-- Base link is the center of the robot's bottom plate -->
+    <link name="base_link">
+      <visual>
+        <origin xyz="0 0 0" rpy="0 0 0" />
         <geometry>
-          <mesh filename="package://m2_description/meshes/dae/body_front_lights_vis.dae" scale="1.0 1.0 1.0"/>
+          <box size="${base_x_size} ${base_y_size} ${base_z_size}"/>
         </geometry>
-        <material name="white_police_light"/>
+        <material name="grey">
+          <color rgba="0.6 0.6 0.6 1"/>
+        </material>
       </visual>
-      <visual name="body_lights_blue_vis">
-        <origin xyz="0.37794 0.18642 0.7649" rpy="0 0 0"/>
+      <collision>
         <geometry>
-          <mesh filename="package://m2_description/meshes/dae/body_lights_blue_vis.dae" scale="1.0 1.0 1.0"/>
-        </geometry>
-        <material name="blue_police_light"/>
-      </visual>
-      <visual name="body_lights_red_vis">
-        <origin xyz="0.37978 -0.18222 0.76491" rpy="0 0 0"/>
-        <geometry>
-          <mesh filename="package://m2_description/meshes/dae/body_lights_red_vis.dae" scale="1.0 1.0 1.0"/>
-        </geometry>
-        <material name="red_police_light"/>
-      </visual>
-      <visual name="body_lights_white_vis">
-        <origin xyz="0.40793 0.00023 0.7689" rpy="0 0 0"/>
-        <geometry>
-          <mesh filename="package://m2_description/meshes/dae/body_lights_white_vis.dae" scale="1.0 1.0 1.0"/>
-        </geometry>
-        <material name="white_police_light"/>
-      </visual>
-      <visual name="body_vis">
-        <origin xyz="0.07415 0.00012 0.24822" rpy="0 0 0"/>
-        <geometry>
-          <mesh filename="package://m2_description/meshes/dae/body_vis.dae" scale="1.0 1.0 1.0"/>
-        </geometry>
-        <material name="body_grey"/>
-      </visual>
-      <visual name="camera_top_vis">
-        <origin xyz="0.11195 0.00142 1.30874" rpy="-1.5708 0 0"/>
-        <geometry>
-          <mesh filename="package://m2_description/meshes/dae/camera_top_vis.dae" scale="1.0 1.0 1.0"/>
-        </geometry>
-        <material name="body_black"/>
-      </visual>
-      <visual name="chassis_vis">
-        <origin xyz="0.01034 -3e-05 0.00065" rpy="0 0 0"/>
-        <geometry>
-          <mesh filename="package://m2_description/meshes/dae/chassis_vis.dae" scale="1.0 1.0 1.0"/>
-        </geometry>
-        <material name="Metal_Bling chrome"/>
-      </visual>
-      <visual name="text_body_vis">
-        <origin xyz="-0.38196 0.00023 0.4187" rpy="0 0 0"/>
-        <geometry>
-          <mesh filename="package://m2_description/meshes/dae/text_body_vis.dae" scale="1.0 1.0 1.0"/>
-        </geometry>
-        <material name="body_black"/>
-      </visual>
-      <visual name="text_front_vis">
-        <origin xyz="-0.38196 0.00023 0.4187" rpy="0 0 0"/>
-        <geometry>
-          <mesh filename="package://m2_description/meshes/dae/text_front_vis.dae" scale="1.0 1.0 1.0"/>
-        </geometry>
-        <material name="body_grey"/>
-      </visual>
-      <collision name="body_col">
-        <origin xyz="0.00514 0.00023 0.42524" rpy="0 0 0"/>
-        <geometry>
-          <box size="2.01448 0.94935 1.16925"/>
-        </geometry>
-      </collision>
-      <collision name="camera_top_col">
-        <origin xyz="0.11195 0.0019 1.25215" rpy="0 0 0"/>
-        <geometry>
-          <cylinder radius="0.06976" length="0.25"/>
-        </geometry>
-      </collision>
-      <collision name="chassis_col">
-        <origin xyz="0.01121 0.00023 0.02431" rpy="0 0 0"/>
-        <geometry>
-          <box size="1.9958 0.72 0.35508"/>
+          <box size="${base_x_size} ${base_y_size} ${base_z_size}"/>
         </geometry>
       </collision>
     </link>
-    <link name="drive_motor_lb">
+    <joint name="base_footprint_joint" type="fixed">
+      <origin xyz="0 0 ${ground_clearance + base_z_size/2}" rpy="0 0 0" />
+      <child link="base_link" />
+      <parent link="base_footprint" />
+    </joint>
+    <!-- Interial link stores the robot's inertial information -->
+    <link name="inertial_link">
       <inertial>
-        <origin xyz="-0.00105 0.08331 0.05321" rpy="0 0 0"/>
-        <mass value="17.0"/>
-        <inertia ixx="0.09492" ixy="6e-05" ixz="8e-05" iyy="0.03042" iyz="-0.00181" izz="0.09704"/>
+        <mass value="340" />
+        <origin xyz="0 0 0" />
+        <inertia ixx="${mass_base/12.0 * (base_y_size*base_y_size + base_z_size*base_z_size)}" ixy="0" ixz="0"
+                 iyy="${mass_base/12.0 * (base_x_size*base_x_size + base_z_size*base_z_size)}" iyz="0"
+                 izz="${mass_base/12.0 * (base_y_size*base_y_size + base_x_size*base_x_size)}" />
       </inertial>
-      <visual name="drive_motor_lb_vis">
-        <origin xyz="0 0 0" rpy="0 0 0"/>
-        <geometry>
-          <mesh filename="package://m2_description/meshes/dae/drive_motor_lb_vis.dae" scale="1.0 1.0 1.0"/>
-        </geometry>
-        <material name="body_black"/>
-      </visual>
-      <collision name="drive_motor_lb_col">
-        <origin xyz="0 0.09943 0.0535" rpy="0 0 0"/>
-        <geometry>
-          <box size="0.129 0.34444 0.107"/>
-        </geometry>
-      </collision>
     </link>
-    <link name="drive_motor_lf">
-      <inertial>
-        <origin xyz="0.00102 0.07894 0.05182" rpy="0 0 0"/>
-        <mass value="17.0"/>
-        <inertia ixx="0.09256" ixy="0" ixz="4e-05" iyy="0.03047" iyz="-0.00143" izz="0.09479"/>
-      </inertial>
-      <visual name="drive_motor_lf_vis">
-        <origin xyz="0 0 0" rpy="0 0 0"/>
-        <geometry>
-          <mesh filename="package://m2_description/meshes/dae/drive_motor_lf_vis.dae" scale="1.0 1.0 1.0"/>
-        </geometry>
-        <material name="body_black"/>
-      </visual>
-      <collision name="drive_motor_lf_col">
-        <origin xyz="0 0.08243 0.0535" rpy="0 0 0"/>
-        <geometry>
-          <box size="0.129 0.31044 0.107"/>
-        </geometry>
-      </collision>
-    </link>
-    <link name="drive_motor_rb">
-      <inertial>
-        <origin xyz="-0.00156 -0.08306 0.05155" rpy="0 0 0"/>
-        <mass value="17.0"/>
-        <inertia ixx="0.0948" ixy="3e-05" ixz="-4e-05" iyy="0.03031" iyz="0.00155" izz="0.09706"/>
-      </inertial>
-      <visual name="drive_motor_rb_vis">
-        <origin xyz="0 0 0" rpy="0 0 0"/>
-        <geometry>
-          <mesh filename="package://m2_description/meshes/dae/drive_motor_rb_vis.dae" scale="1.0 1.0 1.0"/>
-        </geometry>
-        <material name="body_black"/>
-      </visual>
-      <collision name="drive_motor_rb_col">
-        <origin xyz="0 -0.09943 0.0535" rpy="0 0 0"/>
-        <geometry>
-          <box size="0.129 0.34444 0.107"/>
-        </geometry>
-      </collision>
-    </link>
-    <link name="drive_motor_rf">
-      <inertial>
-        <origin xyz="0.00053 -0.08238 0.0526" rpy="0 0 0"/>
-        <mass value="17.0"/>
-        <inertia ixx="0.09367" ixy="0" ixz="4e-05" iyy="0.03055" iyz="0.00168" izz="0.09585"/>
-      </inertial>
-      <visual name="drive_motor_rf_vis">
-        <origin xyz="0 0 0" rpy="0 0 0"/>
-        <geometry>
-          <mesh filename="package://m2_description/meshes/dae/drive_motor_rf_vis.dae" scale="1.0 1.0 1.0"/>
-        </geometry>
-        <material name="body_black"/>
-      </visual>
-      <collision name="drive_motor_rf_col">
-        <origin xyz="0 -0.08243 0.0535" rpy="0 0 0"/>
-        <geometry>
-          <box size="0.129 0.31044 0.107"/>
-        </geometry>
-      </collision>
-    </link>
-    <link name="shock_lb_1">
-      <inertial>
-        <origin xyz="0.05551 0.02184 0" rpy="0 0 0"/>
-        <mass value="0.2"/>
-        <inertia ixx="0.00025" ixy="2e-05" ixz="2e-05" iyy="0.00016" iyz="-0.0001" izz="0.00014"/>
-      </inertial>
-      <visual name="shock_lb_1_vis">
-        <origin xyz="0 0 0" rpy="-0.37525 -1.5708 0"/>
-        <geometry>
-          <mesh filename="package://m2_description/meshes/dae/shock_lb_1_vis.dae" scale="1.0 1.0 1.0"/>
-        </geometry>
-        <material name="Metal_Bling chrome"/>
-      </visual>
-      <collision name="shock_lb_1_col">
-        <origin xyz="0.0564 0.02221 0" rpy="0.37525 -1.5708 0"/>
-        <geometry>
-          <cylinder radius="0.026" length="0.143"/>
-        </geometry>
-      </collision>
-    </link>
-    <link name="shock_lb_2">
-      <inertial>
-        <origin xyz="-0.00989 -0.0039 0" rpy="0 0 0"/>
-        <mass value="0.1"/>
-        <inertia ixx="2e-05" ixy="0" ixz="0" iyy="2e-05" iyz="0" izz="2e-05"/>
-      </inertial>
-      <visual name="shock_lb_2_vis">
-        <origin xyz="0 0 0" rpy="-0.37525 -1.5708 0"/>
-        <geometry>
-          <mesh filename="package://m2_description/meshes/dae/shock_lb_2_vis.dae" scale="1.0 1.0 1.0"/>
-        </geometry>
-        <material name="Metal_Bling chrome"/>
-      </visual>
-      <collision name="shock_lb_2_col">
-        <origin xyz="-0.01732 -0.00682 0" rpy="0.37525 -1.5708 0"/>
-        <geometry>
-          <cylinder radius="0.025" length="0.0588"/>
-        </geometry>
-      </collision>
-    </link>
-    <link name="shock_lf_1">
-      <inertial>
-        <origin xyz="0.05551 0.02184 0" rpy="0 0 0"/>
-        <mass value="0.2"/>
-        <inertia ixx="0.00025" ixy="2e-05" ixz="2e-05" iyy="0.00016" iyz="-0.0001" izz="0.00014"/>
-      </inertial>
-      <visual name="shock_lf_1_vis">
-        <origin xyz="0 0 0" rpy="-0.37525 -1.5708 0"/>
-        <geometry>
-          <mesh filename="package://m2_description/meshes/dae/shock_lf_1_vis.dae" scale="1.0 1.0 1.0"/>
-        </geometry>
-        <material name="Metal_Bling chrome"/>
-      </visual>
-      <collision name="shock_lf_1_col">
-        <origin xyz="0.0564 0.02221 0" rpy="0.37525 -1.5708 0"/>
-        <geometry>
-          <cylinder radius="0.026" length="0.143"/>
-        </geometry>
-      </collision>
-    </link>
-    <link name="shock_lf_2">
-      <inertial>
-        <origin xyz="-0.00989 -0.00389 0" rpy="0 0 0"/>
-        <mass value="0.1"/>
-        <inertia ixx="2e-05" ixy="0" ixz="0" iyy="2e-05" iyz="0" izz="2e-05"/>
-      </inertial>
-      <visual name="shock_lf_2_vis">
-        <origin xyz="0 0 0" rpy="-0.37525 -1.5708 0"/>
-        <geometry>
-          <mesh filename="package://m2_description/meshes/dae/shock_lf_2_vis.dae" scale="1.0 1.0 1.0"/>
-        </geometry>
-        <material name="Metal_Bling chrome"/>
-      </visual>
-      <collision name="shock_lf_2_col">
-        <origin xyz="-0.01732 -0.00682 0" rpy="0.37525 -1.5708 0"/>
-        <geometry>
-          <cylinder radius="0.025" length="0.0588"/>
-        </geometry>
-      </collision>
-    </link>
-    <link name="shock_rb_1">
-      <inertial>
-        <origin xyz="0.05551 -0.02184 0" rpy="0 0 0"/>
-        <mass value="0.2"/>
-        <inertia ixx="0.00025" ixy="-2e-05" ixz="2e-05" iyy="0.00016" iyz="0.0001" izz="0.00014"/>
-      </inertial>
-      <visual name="shock_rb_1_vis">
-        <origin xyz="0 0 0" rpy="-0.37525 -1.5708 0"/>
-        <geometry>
-          <mesh filename="package://m2_description/meshes/dae/shock_rb_1_vis.dae" scale="1.0 1.0 1.0"/>
-        </geometry>
-        <material name="Metal_Bling chrome"/>
-      </visual>
-      <collision name="shock_rb_1_col">
-        <origin xyz="0.0564 -0.02221 0" rpy="-0.37525 -1.5708 0"/>
-        <geometry>
-          <cylinder radius="0.026" length="0.143"/>
-        </geometry>
-      </collision>
-    </link>
-    <link name="shock_rb_2">
-      <inertial>
-        <origin xyz="-0.00989 0.0039 0" rpy="0 0 0"/>
-        <mass value="0.1"/>
-        <inertia ixx="2e-05" ixy="0" ixz="0" iyy="2e-05" iyz="0" izz="2e-05"/>
-      </inertial>
-      <visual name="shock_rb_2_vis">
-        <origin xyz="0 0 0" rpy="-0.37525 -1.5708 0"/>
-        <geometry>
-          <mesh filename="package://m2_description/meshes/dae/shock_rb_2_vis.dae" scale="1.0 1.0 1.0"/>
-        </geometry>
-        <material name="Metal_Bling chrome"/>
-      </visual>
-      <collision name="shock_rb_2_col">
-        <origin xyz="-0.01732 0.00682 0" rpy="-0.37525 -1.5708 0"/>
-        <geometry>
-          <cylinder radius="0.025" length="0.0588"/>
-        </geometry>
-      </collision>
-    </link>
-    <link name="shock_rf_1">
-      <inertial>
-        <origin xyz="0.05551 -0.02184 0" rpy="0 0 0"/>
-        <mass value="0.2"/>
-        <inertia ixx="0.00025" ixy="-2e-05" ixz="2e-05" iyy="0.00016" iyz="0.0001" izz="0.00014"/>
-      </inertial>
-      <visual name="shock_rf_1_vis">
-        <origin xyz="-0.00212 0 0" rpy="-0.37525 -1.5708 0"/>
-        <geometry>
-          <mesh filename="package://m2_description/meshes/dae/shock_rf_1_vis.dae" scale="1.0 1.0 1.0"/>
-        </geometry>
-        <material name="Metal_Bling chrome"/>
-      </visual>
-      <collision name="shock_rf_1_col">
-        <origin xyz="0.0564 -0.02221 0" rpy="-0.37525 -1.5708 0"/>
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