Commit message: adding swerve control robot

File: src/ros_controllers/ackermann_steering_controller/test/common/urdf/ackermann_steering_bot.xacro (robot description, xacro)
@@ -53,26 +53,26 @@
   </joint>
   <!-- joints for ackermann_steering_controller -->
-  <xacro:front_steer name="front" parent="base" radius="${wheel_radius}" thickness="${thickness}"
+  <front_steer name="front" parent="base" radius="${wheel_radius}" thickness="${thickness}"
       length="${length}" width="${width}" axel_offset="${axel_offset}" steer_height="${wheel_radius+steer_offset}">
     <origin xyz="${length/2-axel_offset} 0 0" rpy="${-90 * deg_to_rad} 0 0"/>
-  </xacro:front_steer>
-  <xacro:rear_wheel name="rear" parent="base" radius="${wheel_radius}" thickness="${thickness}">
+  </front_steer>
+  <rear_wheel name="rear" parent="base" radius="${wheel_radius}" thickness="${thickness}">
     <origin xyz="${-length/2+axel_offset} 0 0" rpy="${-90 * deg_to_rad} 0 0"/>
-  </xacro:rear_wheel>
+  </rear_wheel>
   <!-- Wheels -->
-  <xacro:front_wheel_lr name="front_right" parent="base" radius="${wheel_radius}" thickness="${thickness}"
+  <front_wheel_lr name="front_right" parent="base" radius="${wheel_radius}" thickness="${thickness}"
       length="${length}" width="${width}" axel_offset="${axel_offset}" right_left="1" steer_height="${wheel_radius+steer_offset}">
     <origin xyz="${length/2-axel_offset} ${width/2+axel_offset} 0" rpy="${-90 * deg_to_rad} 0 0"/>
-  </xacro:front_wheel_lr>
-  <xacro:front_wheel_lr name="front_left" parent="base" radius="${wheel_radius}" thickness="${thickness}"
+  </front_wheel_lr>
+  <front_wheel_lr name="front_left" parent="base" radius="${wheel_radius}" thickness="${thickness}"
       length="${length}" width="${width}" axel_offset="${axel_offset}" right_left="-1" steer_height="${wheel_radius+steer_offset}">
     <origin xyz="${length/2-axel_offset} ${-width/2-axel_offset} 0" rpy="${-90 * deg_to_rad} 0 0"/>
-  </xacro:front_wheel_lr>
-  <xacro:rear_wheel_lr name="rear_right" parent="base" radius="${wheel_radius}" thickness="${thickness}">
+  </front_wheel_lr>
+  <rear_wheel_lr name="rear_right" parent="base" radius="${wheel_radius}" thickness="${thickness}">
     <origin xyz="${-length/2+axel_offset} ${width/2+axel_offset} 0" rpy="${-90 * deg_to_rad} 0 0"/>
-  </xacro:rear_wheel_lr>
-  <xacro:rear_wheel_lr name="rear_left" parent="base" radius="${wheel_radius}" thickness="${thickness}">
+  </rear_wheel_lr>
+  <rear_wheel_lr name="rear_left" parent="base" radius="${wheel_radius}" thickness="${thickness}">
     <origin xyz="${-length/2+axel_offset} ${-width/2-axel_offset} 0" rpy="${-90 * deg_to_rad} 0 0"/>
-  </xacro:rear_wheel_lr>
+  </rear_wheel_lr>
   <!-- Colour -->
   <gazebo reference="base_link">

File: src/ros_controllers/ackermann_steering_controller/test/common/urdf/ackermann_steering_bot_sphere_wheels.xacro (robot description, xacro)
@@ -53,26 +53,26 @@
   </joint>
   <!-- joints for ackermann_steering_controller -->
-  <xacro:front_steer name="front" parent="base" radius="${wheel_radius}" thickness="${thickness}"
+  <front_steer name="front" parent="base" radius="${wheel_radius}" thickness="${thickness}"
       length="${length}" width="${width}" axel_offset="${axel_offset}" steer_height="${wheel_radius+steer_offset}">
     <origin xyz="${length/2-axel_offset} 0 0" rpy="${-90 * deg_to_rad} 0 0"/>
-  </xacro:front_steer>
-  <xacro:rear_wheel name="rear" parent="base" radius="${wheel_radius}" thickness="${thickness}">
+  </front_steer>
+  <rear_wheel name="rear" parent="base" radius="${wheel_radius}" thickness="${thickness}">
     <origin xyz="${-length/2+axel_offset} 0 0" rpy="${-90 * deg_to_rad} 0 0"/>
-  </xacro:rear_wheel>
+  </rear_wheel>
   <!-- Wheels -->
-  <xacro:front_wheel_lr name="front_right" parent="base" radius="${wheel_radius}" thickness="${thickness}"
+  <front_wheel_lr name="front_right" parent="base" radius="${wheel_radius}" thickness="${thickness}"
       length="${length}" width="${width}" axel_offset="${axel_offset}" right_left="1" steer_height="${wheel_radius+steer_offset}">
     <origin xyz="${length/2-axel_offset} ${width/2+axel_offset} 0" rpy="${-90 * deg_to_rad} 0 0"/>
-  </xacro:front_wheel_lr>
-  <xacro:front_wheel_lr name="front_left" parent="base" radius="${wheel_radius}" thickness="${thickness}"
+  </front_wheel_lr>
+  <front_wheel_lr name="front_left" parent="base" radius="${wheel_radius}" thickness="${thickness}"
       length="${length}" width="${width}" axel_offset="${axel_offset}" right_left="-1" steer_height="${wheel_radius+steer_offset}">
     <origin xyz="${length/2-axel_offset} ${-width/2-axel_offset} 0" rpy="${-90 * deg_to_rad} 0 0"/>
-  </xacro:front_wheel_lr>
-  <xacro:rear_wheel_lr name="rear_right" parent="base" radius="${wheel_radius}" thickness="${thickness}">
+  </front_wheel_lr>
+  <rear_wheel_lr name="rear_right" parent="base" radius="${wheel_radius}" thickness="${thickness}">
     <origin xyz="${-length/2+axel_offset} ${width/2+axel_offset} 0" rpy="${-90 * deg_to_rad} 0 0"/>
-  </xacro:rear_wheel_lr>
-  <xacro:rear_wheel_lr name="rear_left" parent="base" radius="${wheel_radius}" thickness="${thickness}">
+  </rear_wheel_lr>
+  <rear_wheel_lr name="rear_left" parent="base" radius="${wheel_radius}" thickness="${thickness}">
     <origin xyz="${-length/2+axel_offset} ${-width/2-axel_offset} 0" rpy="${-90 * deg_to_rad} 0 0"/>
-  </xacro:rear_wheel_lr>
+  </rear_wheel_lr>
   <!-- Colour -->
   <gazebo reference="base_link">

File: src/ros_controllers/diff_drive_controller/test/diffbot.xacro (robot description, xacro)
@@ -51,10 +51,10 @@
   </joint>
   <!-- Wheels -->
-  <xacro:wheel name="wheel_0" parent="base" radius="${wheel_radius}" thickness="${thickness}">
+  <wheel name="wheel_0" parent="base" radius="${wheel_radius}" thickness="${thickness}">
     <origin xyz="${width/2+axel_offset} 0 0" rpy="${-90 * deg_to_rad} 0 0"/>
-  </xacro:wheel>
-  <xacro:wheel name="wheel_1" parent="base" radius="${wheel_radius}" thickness="${thickness}">
+  </wheel>
+  <wheel name="wheel_1" parent="base" radius="${wheel_radius}" thickness="${thickness}">
     <origin xyz="${-width/2+axel_offset} 0 0" rpy="${-90 * deg_to_rad} 0 0"/>
-  </xacro:wheel>
+  </wheel>
   <!-- Colour -->
   <gazebo reference="base_link">

File: src/ros_controllers/diff_drive_controller/test/diffbot_sphere_wheels.xacro (robot description, xacro)
@@ -50,10 +50,10 @@
   </joint>
   <!-- Wheels -->
-  <xacro:sphere_wheel name="wheel_0" parent="base" radius="${wheel_radius}">
+  <sphere_wheel name="wheel_0" parent="base" radius="${wheel_radius}">
     <origin xyz="${width/2+axel_offset} 0 0" rpy="${-90 * deg_to_rad} 0 0"/>
-  </xacro:sphere_wheel>
-  <xacro:sphere_wheel name="wheel_1" parent="base" radius="${wheel_radius}">
+  </sphere_wheel>
+  <sphere_wheel name="wheel_1" parent="base" radius="${wheel_radius}">
     <origin xyz="${-width/2+axel_offset} 0 0" rpy="${-90 * deg_to_rad} 0 0"/>
-  </xacro:sphere_wheel>
+  </sphere_wheel>
   <!-- Colour -->
   <gazebo reference="base_link">

File: src/ros_controllers/diff_drive_controller/test/diffbot_square_wheels.xacro (robot description, xacro)
@@ -50,10 +50,10 @@
   </joint>
   <!-- Wheels -->
-  <xacro:square_wheel name="wheel_0" parent="base" radius="${wheel_radius}">
+  <square_wheel name="wheel_0" parent="base" radius="${wheel_radius}">
     <origin xyz="${width/2+axel_offset} 0 0" rpy="${-90 * deg_to_rad} 0 0"/>
-  </xacro:square_wheel>
-  <xacro:square_wheel name="wheel_1" parent="base" radius="${wheel_radius}">
+  </square_wheel>
+  <square_wheel name="wheel_1" parent="base" radius="${wheel_radius}">
     <origin xyz="${-width/2+axel_offset} 0 0" rpy="${-90 * deg_to_rad} 0 0"/>
-  </xacro:square_wheel>
+  </square_wheel>
   <!-- Colour -->
   <gazebo reference="base_link">

File: src/ros_controllers/diff_drive_controller/test/skidsteerbot.xacro (robot description, xacro)
@@ -52,22 +52,22 @@
   </joint>
   <!-- Wheels -->
-  <xacro:wheel name="wheel_0" parent="base" radius="${wheel_radius}" thickness="${thickness}">
+  <wheel name="wheel_0" parent="base" radius="${wheel_radius}" thickness="${thickness}">
     <origin xyz="${width/2+axel_offset} ${y_offset} 0" rpy="${-90 * deg_to_rad} 0 0"/>
-  </xacro:wheel>
-  <xacro:wheel name="wheel_1" parent="base" radius="${wheel_radius}" thickness="${thickness}">
+  </wheel>
+  <wheel name="wheel_1" parent="base" radius="${wheel_radius}" thickness="${thickness}">
     <origin xyz="${width/2+axel_offset} 0 0" rpy="${-90 * deg_to_rad} 0 0"/>
-  </xacro:wheel>
-  <xacro:wheel name="wheel_2" parent="base" radius="${wheel_radius}" thickness="${thickness}">
+  </wheel>
+  <wheel name="wheel_2" parent="base" radius="${wheel_radius}" thickness="${thickness}">
     <origin xyz="${width/2+axel_offset} ${-y_offset} 0" rpy="${-90 * deg_to_rad} 0 0"/>
-  </xacro:wheel>
-  <xacro:wheel name="wheel_3" parent="base" radius="${wheel_radius}" thickness="${thickness}">
+  </wheel>
+  <wheel name="wheel_3" parent="base" radius="${wheel_radius}" thickness="${thickness}">
     <origin xyz="${-width/2+axel_offset} ${y_offset} 0" rpy="${-90 * deg_to_rad} 0 0"/>
-  </xacro:wheel>
-  <xacro:wheel name="wheel_4" parent="base" radius="${wheel_radius}" thickness="${thickness}">
+  </wheel>
+  <wheel name="wheel_4" parent="base" radius="${wheel_radius}" thickness="${thickness}">
     <origin xyz="${-width/2+axel_offset} 0 0" rpy="${-90 * deg_to_rad} 0 0"/>
-  </xacro:wheel>
-  <xacro:wheel name="wheel_5" parent="base" radius="${wheel_radius}" thickness="${thickness}">
+  </wheel>
+  <wheel name="wheel_5" parent="base" radius="${wheel_radius}" thickness="${thickness}">
     <origin xyz="${-width/2+axel_offset} ${-y_offset} 0" rpy="${-90 * deg_to_rad} 0 0"/>
-  </xacro:wheel>
+  </wheel>
   <!-- Colour -->
   <gazebo reference="base_link">

File: src/ros_controllers/four_wheel_steering_controller/test/urdf/chassis.xacro (robot description, xacro)
@@ -3,9 +3,9 @@
   <!-- Base Properties -->
   <xacro:property name="mass_base" value="340" />
-  <xacro:property name="base_x_size" value="0.66000" />
+  <xacro:property name="base_x_size" value="1.66000" />
   <xacro:property name="base_y_size" value="0.60000" />
-  <xacro:property name="base_z_size" value="0.16000" />
-  <xacro:property name="wheelbase" value="1.66" />
-  <xacro:property name="track" value="1.2" />
+  <xacro:property name="base_z_size" value="0.66000" />
+  <xacro:property name="wheelbase" value="1.9" />
+  <xacro:property name="track" value="1.1" />
   <xacro:macro name="chassis">
     <!-- Base footprint is on the ground under the robot -->
@@ -51,124 +51,4 @@
       <child link="inertial_link" />
     </joint>
-    <material name="LiDAR_grey">
-      <color rgba="0.59608 0.59608 0.59608 1.0"/>
-    </material>
-    <material name="Metal_Bling chrome">
-      <color rgba="0.8 0.8 0.82431 1.0"/>
-    </material>
-    <material name="Synth_Tyre rubber">
-      <color rgba="0.01678 0.01212 0.01212 1.0"/>
-    </material>
-    <material name="blue_police_light">
-      <color rgba="0 0 1.0 1.0"/>
-    </material>
-    <material name="body_black">
-      <color rgba="0.10594 0.10594 0.10594 1.0"/>
-    </material>
-    <material name="body_grey">
-      <color rgba="0.96 0.96 0.96 1.0"/>
-    </material>
-    <material name="red_police_light">
-      <color rgba="1.0 0 0 1.0"/>
-    </material>
-    <material name="white_police_light">
-      <color rgba="1.0 1.0 1.0 1.0"/>
-    </material>
-    <material name="dummy_mat">
-      <color rgba="0.4 0.4 0.4 1.0"/>
-    </material>
-    <link name="chassis_m2">
-      <inertial>
-        <origin xyz="0.08838 -0.00198 0.17552" rpy="0 0 0"/>
-        <mass value="200.0"/>
-        <inertia ixx="24.43942" ixy="-3.57208" ixz="-2.64293" iyy="116.11656" iyz="0.10486" izz="111.43803"/>
-      </inertial>
-      <visual name="body_front_lights_vis">
-        <origin xyz="0.98421 0.00023 0.09713" rpy="0 0 0"/>
-        <geometry>
-          <mesh filename="package://m2_description/meshes/dae/body_front_lights_vis.dae" scale="1.0 1.0 1.0"/>
-        </geometry>
-        <material name="white_police_light"/>
-      </visual>
-      <visual name="body_lights_blue_vis">
-        <origin xyz="0.37794 0.18642 0.7649" rpy="0 0 0"/>
-        <geometry>
-          <mesh filename="package://m2_description/meshes/dae/body_lights_blue_vis.dae" scale="1.0 1.0 1.0"/>
-        </geometry>
-        <material name="blue_police_light"/>
-      </visual>
-      <visual name="body_lights_red_vis">
-        <origin xyz="0.37978 -0.18222 0.76491" rpy="0 0 0"/>
-        <geometry>
-          <mesh filename="package://m2_description/meshes/dae/body_lights_red_vis.dae" scale="1.0 1.0 1.0"/>
-        </geometry>
-        <material name="red_police_light"/>
-      </visual>
-      <visual name="body_lights_white_vis">
-        <origin xyz="0.40793 0.00023 0.7689" rpy="0 0 0"/>
-        <geometry>
-          <mesh filename="package://m2_description/meshes/dae/body_lights_white_vis.dae" scale="1.0 1.0 1.0"/>
-        </geometry>
-        <material name="white_police_light"/>
-      </visual>
-      <visual name="body_vis">
-        <origin xyz="0.07415 0.00012 0.24822" rpy="0 0 0"/>
-        <geometry>
-          <mesh filename="package://m2_description/meshes/dae/body_vis.dae" scale="1.0 1.0 1.0"/>
-        </geometry>
-        <material name="body_grey"/>
-      </visual>
-      <visual name="camera_top_vis">
-        <origin xyz="0.11195 0.00142 1.30874" rpy="-1.5708 0 0"/>
-        <geometry>
-          <mesh filename="package://m2_description/meshes/dae/camera_top_vis.dae" scale="1.0 1.0 1.0"/>
-        </geometry>
-        <material name="body_black"/>
-      </visual>
-      <visual name="chassis_vis">
-        <origin xyz="0.01034 -3e-05 0.00065" rpy="0 0 0"/>
-        <geometry>
-          <mesh filename="package://m2_description/meshes/dae/chassis_vis.dae" scale="1.0 1.0 1.0"/>
-        </geometry>
-        <material name="Metal_Bling chrome"/>
-      </visual>
-      <visual name="text_body_vis">
-        <origin xyz="-0.38196 0.00023 0.4187" rpy="0 0 0"/>
-        <geometry>
-          <mesh filename="package://m2_description/meshes/dae/text_body_vis.dae" scale="1.0 1.0 1.0"/>
-        </geometry>
-        <material name="body_black"/>
-      </visual>
-      <visual name="text_front_vis">
-        <origin xyz="-0.38196 0.00023 0.4187" rpy="0 0 0"/>
-        <geometry>
-          <mesh filename="package://m2_description/meshes/dae/text_front_vis.dae" scale="1.0 1.0 1.0"/>
-        </geometry>
-        <material name="body_grey"/>
-      </visual>
-      <collision name="body_col">
-        <origin xyz="0.00514 0.00023 0.42524" rpy="0 0 0"/>
-        <geometry>
-          <box size="2.01448 0.94935 1.16925"/>
-        </geometry>
-      </collision>
-      <collision name="camera_top_col">
-        <origin xyz="0.11195 0.0019 1.25215" rpy="0 0 0"/>
-        <geometry>
-          <cylinder radius="0.06976" length="0.25"/>
-        </geometry>
-      </collision>
-      <collision name="chassis_col">
-        <origin xyz="0.01121 0.00023 0.02431" rpy="0 0 0"/>
-        <geometry>
-          <box size="1.9958 0.72 0.35508"/>
-        </geometry>
-      </collision>
-    </link>
-    <joint name="base_footprint_to_chassis" type="fixed">
-      <origin xyz="0 0 0" rpy="0 0 0"/>
-      <parent link="base_link"/>
-      <child link="chassis_m2"/>
-    </joint>
   </xacro:macro>
 </robot>

File: src/ros_controllers/four_wheel_steering_controller/test/urdf/four_wheel_steering.urdf.xacro (robot description, xacro)
@@ -7,5 +7,5 @@
   <xacro:property name="ground_clearance" value="0.19" />
   <xacro:property name="wheel_x_offset" value="0.0" />
-  <xacro:property name="wheel_y_offset" value="0.1" />
+  <xacro:property name="wheel_y_offset" value="0.05" />
   <xacro:chassis/>
   <!-- Wheel macros -->

File: src/ros_controllers/four_wheel_steering_controller/test/urdf/wheel.xacro (robot description, xacro)
@@ -3,6 +3,6 @@
   <!--<xacro:property name="M_PI" default="3.14159"/>-->
   <!-- Wheel Properties -->
-  <xacro:property name="wheel_length" value="0.18" />
-  <xacro:property name="wheel_radius" value="0.22" />
+  <xacro:property name="wheel_length" value="0.1" />
+  <xacro:property name="wheel_radius" value="0.28" />
   <xacro:property name="mass_wheel" value="5.0" />
   <xacro:macro name="wheel" params="wheel_prefix parent_link left_right *joint_origin">
@@ -38,6 +38,6 @@
 		</link>
 		<gazebo reference="${wheel_prefix}_wheel_link">
-			<mu1 value="0.5"/>
-			<mu2 value="0.5"/>
+			<mu1 value="1.0"/>
+			<mu2 value="1.0"/>
 			<kp value="10000000.0" />
 			<kd value="1.0" />
