Commit message: add 360move, crub mood

File: src/ros_controllers/swerve_controller/test/urdf/swervebot.xacro (robot description, xacro)
@@ -560,5 +560,5 @@
       <child link="drive_motor_lb"/>
       <axis xyz="0 0 1.0"/>
-      <limit lower="-0.575958653" upper="1.151917306" effort="10.0" velocity="3000.0"/>
+      <limit lower="-0.575958653" upper="1.151917306" effort="100.0" velocity="3000.0"/>
       <!-- lower and upper limits => rad -->
       <!-- effort => N.m -->
@@ -571,6 +571,6 @@
       <parent link="steering_strut_lf"/>
       <child link="drive_motor_lf"/>
-      <axis xyz="0 0 -1.0"/>
-      <limit lower="-0.575958653" upper="1.151917306" effort="10.0" velocity="3000.0"/>
+      <axis xyz="0 0 1.0"/>
+      <limit lower="-0.575958653" upper="1.151917306" effort="100.0" velocity="3000.0"/>
       <!-- lower and upper limits => rad -->
       <!-- effort => N.m -->
@@ -583,6 +583,6 @@
       <parent link="steering_strut_rb"/>
       <child link="drive_motor_rb"/>
-      <axis xyz="0 0 -1.0"/>
-      <limit lower="-0.575958653" upper="1.151917306" effort="10.0" velocity="3000.0"/>
+      <axis xyz="0 0 1.0"/>
+      <limit lower="-0.575958653" upper="1.151917306" effort="100.0" velocity="3000.0"/>
       <!-- lower and upper limits => rad -->
       <!-- effort => N.m -->
@@ -596,5 +596,5 @@
       <child link="drive_motor_rf"/>
       <axis xyz="0 0 1.0"/>
-      <limit lower="-0.575958653" upper="1.151917306" effort="10.0" velocity="3000.0"/>
+      <limit lower="-0.575958653" upper="1.151917306" effort="100.0" velocity="3000.0"/>
       <!-- lower and upper limits => rad -->
       <!-- effort => N.m -->
@@ -690,6 +690,6 @@
       <parent link="drive_motor_lb"/>
       <child link="wheel_lb"/>
-      <axis xyz="0 -1.0 0"/>
-      <limit effort="200.0" velocity="2000.0"/>
+      <axis xyz="0 1.0 0"/>
+      <limit effort="2000.0" velocity="20000.0"/>
       <!-- effort = ? (0.5 stall torque) -->
       <!-- effort => N.m -->
@@ -700,6 +700,6 @@
       <parent link="drive_motor_lf"/>
       <child link="wheel_lf"/>
-      <axis xyz="0 -1.0 0"/>
-      <limit effort="200.0" velocity="2000.0"/>
+      <axis xyz="0 1.0 0"/>
+      <limit effort="2000.0" velocity="20000.0"/>
       <!-- effort = ? (0.5 stall torque) -->
       <!-- effort => N.m -->
@@ -710,6 +710,6 @@
       <parent link="drive_motor_rb"/>
       <child link="wheel_rb"/>
-      <axis xyz="0 -1.0 0"/>
-      <limit effort="200.0" velocity="2000.0"/>
+      <axis xyz="0 1.0 0"/>
+      <limit effort="2000.0" velocity="20000.0"/>
       <!-- effort = ? (0.5 stall torque) -->
       <!-- effort => N.m -->
@@ -720,6 +720,6 @@
       <parent link="drive_motor_rf"/>
       <child link="wheel_rf"/>
-      <axis xyz="0 -1.0 0"/>
-      <limit effort="200.0" velocity="2000.0"/>
+      <axis xyz="0 1.0 0"/>
+      <limit effort="2000.0" velocity="20000.0"/>
       <!-- effort = ? (0.5 stall torque) -->
       <!-- effort => N.m -->
